File: VGA-Breakout/VGA-Breakout.kicad_pcb (KiCad board)
At the start: 2 copper layers, 38.7 x 69.2 mm, 3 parts, among them J1 DE15_Receptacle_HighDensity, J2 Conn_02x08_Top_Bottom, J3 Conn_02x04_Odd_Even

Commit message: Corerect URL.
Other:
- board text added: "VGA Breakout Board Revision 1 ©2024 Dieter Baron github.com/T-Pau/Connector-Breakout-Boards"
- board text removed: "JLCJLCJLCJLC"
- board text removed: "VGA Breakout Board Revision 1 ©2024 Dieter Baron github.com/T-Pau/VGA-Breakout"
