File: DIN-6/DIN-6.kicad_pcb (KiCad board)
At the start: 2 copper layers, 60 x 59.5 mm, 3 parts, among them J1 Socket, J2 Pins, J3 Breakout

Commit message: Begin SCART breakout board.
Other:
- board text added: "DIN-6 Breakout Board Revision 1 ©2025 Dieter Baron github.com/T-Pau/Connector-Breakout-Boards"
- board text removed: "DIN-6 Breakout Board ©2025 Dieter Baron github.com/T-Pau/Connector-Breakout-Boards"
